Commit message: Fixed elevator use with complex robot models

File: smrr_description/urdf/smrr_description.urdf (robot description, URDF)
Before this commit: robot smrr, 15 links, 14 joints
Links:
- link back_caster: geometry collision sphere radius=0.05; visual sphere radius=0.05
- link base_link: mass 28.2797481488828 -> 8.2797481488828
- link front_caster: geometry collision sphere radius=0.05; visual sphere radius=0.05

Commit message: Reduced impulses in robot within the elevator

File: smrr_description/urdf/smrr_description.urdf (robot description, URDF)
Before this commit: robot smrr, 15 links, 14 joints
Links:
- link left_wheel: geometry collision cylinder length=0.05 radius=0.08; visual cylinder length=0.05 radius=0.08
- link right_wheel: geometry collision cylinder length=0.05 radius=0.08; visual cylinder length=0.05 radius=0.08

Commit message: Updated maps and robot stability

File: smrr_description/urdf/smrr_description.urdf (robot description, URDF)
Before this commit: robot smrr, 15 links, 14 joints
Links:
- link left_wheel: geometry collision cylinder length=0.05 radius=0.081; visual cylinder length=0.05 radius=0.081
- link right_wheel: geometry collision cylinder length=0.05 radius=0.081; visual cylinder length=0.05 radius=0.081
